Commit message: added many things

File: gokul_description/urdf/gokul.xacro (robot description, xacro)
@@ -3,5 +3,7 @@
 <xacro:include filename="$(find gokul_description)/urdf/materials.xacro" />
 <xacro:include filename="$(find gokul_description)/urdf/gokul.trans" />
-<xacro:include filename="$(find gokul_description)/urdf/gokul.gazebo" />
+<xacro:include filename="$(find gokul_description)/gazebo/gokul_materials.gazebo" />
+<xacro:include filename="$(find gokul_description)/gazebo/gokul_physics.gazebo" />
+<xacro:include filename="$(find gokul_description)/gazebo/gokul_plugins.gazebo" />
 <link name="base_link">
   <inertial>
@@ -15,5 +17,5 @@
       <mesh filename="package://gokul_description/meshes/base_link.stl" scale="0.001 0.001 0.001"/>
     </geometry>
-    <material name="silver"/>
+    <material name="blue"/>
   </visual>
   <collision>
@@ -248,5 +250,5 @@
   <parent link="motor_rf_1"/>
   <child link="wheel_rf_1"/>
-  <axis xyz="-0.0 -1.0 0.0"/>
+  <axis xyz="-0.0 1.0 0.0"/>
 </joint>
 <joint name="rev_rb" type="continuous">
@@ -254,5 +256,5 @@
   <parent link="motor_br_1"/>
   <child link="wheel_rb_1"/>
-  <axis xyz="0.0 -1.0 0.0"/>
+  <axis xyz="0.0 1.0 0.0"/>
 </joint>
 <joint name="rev_lf" type="continuous">

File: gokul_description/urdf/materials.xacro (robot description, xacro)
@@ -4,3 +4,6 @@
   <color rgba="0.700 0.700 0.700 1.000"/>
 </material>
+<material name="blue">
+  <color rgba="0.4117 0.733 1.000 1.000"/>
+</material>
 </robot>
